File: Design/Design.kicad_pcb (KiCad board)
At the start: 2 copper layers, 30.5 x 59.7 mm, 20 parts, among them J1 SensorIn, J2 ESP8266 L, J3 ESP8266 R, J4 sensorOut, J5 Joystick, J6 Conn_01x02, J7 buttons, Q1 BC337, Q2 BC337

Commit message: pcb design
Routing:
- added copper zone on F.Cu, net G
Changed lines of the file:
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@@
   (segment (start 92.805 102.965) (end 92.805 97.885) (width 0.25) (layer "F.Cu") (net 40))
   (segment (start 92.805 97.885) (end 91.44 96.52) (width 0.25) (layer "F.Cu") (net 40))
+  (zone (net 4) (net_name "G") (layer "F.Cu") (hatch edge 0.508)
+    (connect_pads (clearance 0.508))
+    (min_thickness 0.254) (filled_areas_thickness no)
+    (fill yes (thermal_gap 0.508) (thermal_bridge_width 0.508))
+    (polygon
+      (pts
+        (xy 105.41 73.66)
+        (xy 105.41 109.22)
+        (xy 71.12 109.22)
+        (xy 71.12 46.99)
+        (xy 105.41 46.99)
+      )
+    )
+  )
   (zone (net 4) (net_name "G") (layer "B.Cu") (hatch edge 0.508)
     (connect_pads (clearance 0.508))
